Commit message: Editing odometry

File: hunter_se_description/models/xacro/hunter_gazebo.xacro (robot description, xacro)
@@ -1,49 +1,4 @@
 <?xml version="1.0"?>
 <robot name="hunter_se_gazebo" xmlns:xacro="http://wiki.ros.org/xacro">
-    <xacro:macro name="ackermann_control">
-        <gazebo>
-            <!-- <plugin name="gazebo_ros_ackermann_drive" filename="libgazebo_ros_ackermann_drive.so">
-                <update_rate>100.0</update_rate>
-                <ros>
-                    <namespace>${robot_namespace}</namespace>
-                    <remapping>odom:=wheel/odometry</remapping>
-                    <remapping>distance:=wheel/distance</remapping>
-                </ros>
-                <initial_orientation_as_reference>true</initial_orientation_as_reference>
-                <front_right_joint>front_right_wheel_joint</front_right_joint>
-                <front_left_joint>front_left_wheel_joint</front_left_joint>
-                <rear_right_joint>rear_right_wheel_joint</rear_right_joint>
-                <rear_left_joint>rear_left_wheel_joint</rear_left_joint>
-                <left_steering_joint>front_left_steer_joint</left_steering_joint>
-                <right_steering_joint>front_right_steer_joint</right_steering_joint>
-                <steering_wheel_joint>center_steer_joint</steering_wheel_joint>
-                <wheel_base>${wheelbase}</wheel_base>
-                <wheel_separation>${wheel_separation}</wheel_separation>
-                <wheel_radius>${wheel_radius}</wheel_radius>
-                <kingpin_width>${2* steering_axle_y_offset}</kingpin_width>
-                <steering_limit>${max_steer}</steering_limit>
-                <min_velocity>-5</min_velocity>
-                <max_velocity>10</max_velocity>
-                <min_aceleration>-2.5</min_aceleration>
-                <max_acceleration>3.5</max_acceleration>
-                <frameID>hunter_se/base_link</frameID>
-                <publish_odom>true</publish_odom>
-                <publish_odom_tf>true</publish_odom_tf>
-                <publish_wheel_tf>true</publish_wheel_tf>
-                <publish_distance>false</publish_distance>
-                <odometry_frame>odom</odometry_frame>
-                <robot_base_frame>base_link</robot_base_frame>
-            </plugin> -->
-            <!-- <plugin name="gazebo_ros_joint_state_publisher"
-                filename="libgazebo_ros_joint_state_publisher.so">
-                <ros>
-                    <namespace>${robot_namespace}</namespace>
-                </ros>
-                <update_rate>20</update_rate>
-                <joint_name>front_right_wheel_joint</joint_name>
-                <joint_name>front_left_wheel_joint</joint_name>
-            </plugin> -->
-        </gazebo>
-    </xacro:macro>
     <xacro:macro name="steering_control"
         params="
@@ -75,3 +30,109 @@
         </joint>
     </xacro:macro>
+    <xacro:macro name="ackermann_odometry">
+        <gazebo>
+            <plugin name="gazebo_ros_ackermann_drive" filename="libgazebo_ros_ackermann_drive.so">
+                <update_rate>100.0</update_rate>
+                <ros>
+                    <namespace>${robot_namespace}</namespace>
+                    <remapping>odom:=wheel_odom</remapping>
+                    <remapping>distance:=wheel/distance</remapping>
+                </ros>
+                <front_left_joint>front_left_wheel_joint</front_left_joint>
+                <front_right_joint>front_right_wheel_joint</front_right_joint>
+                <rear_left_joint>rear_left_wheel_joint</rear_left_joint>
+                <rear_right_joint>rear_right_wheel_joint</rear_right_joint>
+                <left_steering_joint>front_left_steer_joint</left_steering_joint>
+                <right_steering_joint>front_right_steer_joint</right_steering_joint>
+                <!-- <steering_wheel_joint>center_steer_joint</steering_wheel_joint> -->
+                <max_steer>0.690</max_steer>
+                <max_speed>15</max_speed>
+                <left_steering_pid_gain>1500 0 1</left_steering_pid_gain>
+                <left_steering_i_range>0 0</left_steering_i_range>
+                <right_steering_pid_gain>1500 0 1</right_steering_pid_gain>
+                <right_steering_i_range>0 0</right_steering_i_range>
+                <linear_velocity_pid_gain>1000 0 1</linear_velocity_pid_gain>
+                <linear_velocity_i_range>0 0</linear_velocity_i_range>
+                <publish_odom>true</publish_odom>
+                <publish_odom_tf>false</publish_odom_tf>
+                <publish_wheel_tf>false</publish_wheel_tf>
+                <publish_distance>false</publish_distance>
+                <odometry_frame>wheel_odom</odometry_frame>
+                <robot_base_frame>base_link</robot_base_frame>
+            </plugin>
+        </gazebo>
+    </xacro:macro>
+    <xacro:macro name="imu" params="name parent">
+        <link name="${name}" />
+        <joint name="${name}_joint" type="fixed">
+            <parent link="${parent}" />
+            <child link="${name}" />
+            <origin xyz="0 0 0" rpy="0 0 0" />
+        </joint>
+        <gazebo reference="${name}">
+            <sensor name="imu_sensor" type="imu">
+                <plugin filename="libgazebo_ros_imu_sensor.so" name="imu_plugin">
+                    <ros>
+                        <remapping>~/out:=imu</remapping>
+                    </ros>
+                </plugin>
+                <always_on>true</always_on>
+                <update_rate>100</update_rate>
+                <imu>
+                    <angular_velocity>
+                        <x>
+                            <noise type="gaussian">
+                                <mean>0.0</mean>
+                                <stddev>2e-4</stddev>
+                                <bias_mean>0.0000075</bias_mean>
+                                <bias_stddev>0.0000008</bias_stddev>
+                            </noise>
+                        </x>
+                        <y>
+                            <noise type="gaussian">
+                                <mean>0.0</mean>
+                                <stddev>2e-4</stddev>
+                                <bias_mean>0.0000075</bias_mean>
+                                <bias_stddev>0.0000008</bias_stddev>
+                            </noise>
+                        </y>
+                        <z>
+                            <noise type="gaussian">
+                                <mean>0.0</mean>
+                                <stddev>2e-4</stddev>
+                                <bias_mean>0.0000075</bias_mean>
+                                <bias_stddev>0.0000008</bias_stddev>
+                            </noise>
+                        </z>
+                    </angular_velocity>
+                    <linear_acceleration>
+                        <x>
+                            <noise type="gaussian">
+                                <mean>0.0</mean>
+                                <stddev>1.7e-2</stddev>
+                                <bias_mean>0.1</bias_mean>
+                                <bias_stddev>0.001</bias_stddev>
+                            </noise>
+                        </x>
+                        <y>
+                            <noise type="gaussian">
+                                <mean>0.0</mean>
+                                <stddev>1.7e-2</stddev>
+                                <bias_mean>0.1</bias_mean>
+                                <bias_stddev>0.001</bias_stddev>
+                            </noise>
+                        </y>
+                        <z>
+                            <noise type="gaussian">
+                                <mean>0.0</mean>
+                                <stddev>1.7e-2</stddev>
+                                <bias_mean>0.1</bias_mean>
+                                <bias_stddev>0.001</bias_stddev>
+                            </noise>
+                        </z>
+                    </linear_acceleration>
+                </imu>
+            </sensor>
+        </gazebo>
+    </xacro:macro>
 </robot>

File: hunter_se_description/models/xacro/hunter_se.xacro (robot description, xacro)
@@ -61,5 +61,5 @@
     <xacro:hunter_steer name="front_right" reflect="-1" rotation="${pi/2}" />
     <xacro:hunter_steer name="front_left" reflect="1" rotation="${-pi/2}" />
-    <link name="center_steer_link">
+    <!-- <link name="center_steer_link">
         <collision>
             <origin xyz="0 0 0" rpy="0 0 0" />
@@ -82,8 +82,9 @@
         <axis xyz="0 0 1" rpy="0 0 0" />
         <limit lower="${-max_steer}" upper="${max_steer}" effort="10" velocity="5" />
-    </joint>
+    </joint> -->
     <xacro:hunter_motors name="rear_right" reflect="-1" rotation="${-pi/2}" />
     <xacro:hunter_motors name="rear_left" reflect="1" rotation="${pi/2}" />
-    <xacro:ackermann_control />
+    <xacro:ackermann_odometry />
+    <xacro:imu name="IMU" parent="base_link" />
      <ros2_control name="GazeboSystem" type="system">
         <hardware>

Commit message: Fixed Ackermann wheel eqns

File: hunter_se_description/models/xacro/hunter_gazebo.xacro (robot description, xacro)
@@ -45,5 +45,5 @@
                 <left_steering_joint>front_left_steer_joint</left_steering_joint>
                 <right_steering_joint>front_right_steer_joint</right_steering_joint>
-                <!-- <steering_wheel_joint>center_steer_joint</steering_wheel_joint> -->
+                <steering_wheel_joint>center_steer_joint</steering_wheel_joint>
                 <max_steer>0.690</max_steer>
                 <max_speed>15</max_speed>

File: hunter_se_description/models/xacro/hunter_motors.xacro (robot description, xacro)
@@ -11,14 +11,25 @@
             </visual>
             <collision>
-                <origin xyz="0 0 0" rpy="1.57 0 0" />
+                <!-- <origin xyz="0 0 0" rpy="1.57 0 0" /> -->
+                <origin xyz="0 ${reflect * -0.065} 0" rpy="0 0 ${rotation}" />
                 <geometry>
-                    <cylinder radius="${wheel_radius}" length="${wheel_length}" />
+                    <mesh filename="package://hunter_se_description/models/meshes/rear_wheel.dae" />
+                    <!-- <cylinder radius="${wheel_radius}" length="${wheel_length}" /> -->
                 </geometry>
             </collision>
             <inertial>
-                <mass value="0.5" />
+                <mass value="1.0" />
                 <origin xyz="0 0 0" />
-                <inertia ixx="0.022" ixy="0" ixz="0" iyy="0.022" iyz="0" izz="0.0378" />
+                <inertia ixx="0.006864" ixy="0.0" ixz="0.0" iyy="0.012106" iyz="0.0" izz="0.006864" />
+                <!-- <inertia ixx="0.22" ixy="0.02" ixz="0.02" iyy="0.22" iyz="0.02" izz="0.378" /> -->
             </inertial>
+            <surface>
+                <friction>
+                    <ode>
+                        <mu>1.0</mu>
+                        <mu2>1.0</mu2>
+                    </ode>
+                </friction>
+            </surface>
         </link>
         <joint name="${name}_wheel_joint" type="continuous">
@@ -31,5 +42,5 @@
         <gazebo reference="${name}_wheel_link">
             <mu1 value="1.0" />
-            <mu2 value="2.0" />
+            <mu2 value="1.0" />
             <kp value="10000000.0" />
             <kd value="1.0" />

File: hunter_se_description/models/xacro/hunter_se.xacro (robot description, xacro)
@@ -36,40 +36,36 @@
         </visual>
         <collision>
-            <origin xyz="0 0 -0.05" rpy="0 0 0" />
+            <origin xyz="0 0 0" rpy="0 0 0" />
             <geometry>
-                <box size="${base_x_size} ${base_y_size} ${base_z_size}" />
+                <mesh
+                    filename="package://hunter_se_description/models/meshes/hunter_body.dae" />
             </geometry>
         </collision>
-    </link>
-    <link name="inertial_link">
         <inertial>
-            <mass value="24.73" />
-            <origin xyz="0.015 0.00 0.0" />
-            <inertia ixx="0.12321"
-                ixy="2.512E-06"
-                ixz="4.801E-03"
-                iyy="0.219144"
-                iyz="1.033E-05"
-                izz="0.3136" />
+            <mass value="38" />
+            <origin xyz="0.050 0.00 -0.075" />
+            <!-- <inertia ixx="2.0533" ixy="0.0" ixz="0.0" iyy="2.56993" iyz="0.0" izz="0.69606" /> -->
+            <inertia ixx="0.65" ixy="0.0" ixz="0.0" iyy="2.75" iyz="0.0" izz="3.0" />
         </inertial>
     </link>
-    <joint name="inertial_joint" type="fixed">
-        <origin xyz="0 0 0" rpy="0 0 0" />
-        <parent link="base_link" />
-        <child link="inertial_link" />
+    <link name="base_footprint"/>
+    <joint name="base_joint" type="fixed">
+        <origin xyz="0 0 0.250" rpy="0 0 0" />
+        <parent link="base_footprint" />
+        <child link="base_link" />
     </joint>
     <xacro:hunter_steer name="front_right" reflect="-1" rotation="${pi/2}" />
     <xacro:hunter_steer name="front_left" reflect="1" rotation="${-pi/2}" />
-    <!-- <link name="center_steer_link">
-        <collision>
+    <link name="center_steer_link">
+        <!-- <collision>
             <origin xyz="0 0 0" rpy="0 0 0" />
             <geometry>
                 <cylinder radius="${0.04}" length="${0.06}" />
             </geometry>
-        </collision>
+        </collision> -->
         <inertial>
-            <mass value="0.5" />
-            <origin xyz="0 0 0" />
-            <inertia ixx="0.01" ixy="0" ixz="0" iyy="0.01" iyz="0" izz="0.01" />
+            <mass value="0.25" />
+            <origin xyz="0 0 0" rpy="0 0 0" />
+            <inertia ixx="0.000105" ixy="0.0" ixz="0.0" iyy="0.00002" iyz="0.0" izz="0.000105" />
         </inertial>
     </link>
@@ -80,16 +76,20 @@
             xyz="${steering_axle_x_offset} 0 ${steering_axle_z_offset}"
             rpy="0 0 0" />
-        <axis xyz="0 0 1" rpy="0 0 0" />
-        <limit lower="${-max_steer}" upper="${max_steer}" effort="10" velocity="5" />
-    </joint> -->
+        <axis xyz="0 0 1" />
+        <limit lower="${-max_steer}" upper="${max_steer}" effort="100" velocity="5.0" />
+    </joint>
     <xacro:hunter_motors name="rear_right" reflect="-1" rotation="${-pi/2}" />
     <xacro:hunter_motors name="rear_left" reflect="1" rotation="${pi/2}" />
-    <xacro:ackermann_odometry />
+    <!-- <xacro:ackermann_odometry /> -->
     <xacro:imu name="IMU" parent="base_link" />
-     <ros2_control name="GazeboSystem" type="system">
+    <ros2_control name="GazeboSystem" type="system">
         <hardware>
             <plugin>gazebo_ros2_control/GazeboSystem</plugin>
             <robotNamespace>${robot_namespace}</robotNamespace>
         </hardware>
+        <xacro:steering_control
+            name="center"
+            steer_limlow="${-max_steer}"
+            steer_limhigh="${max_steer}" />
         <xacro:steering_control
             name="front_right"

File: hunter_se_description/models/xacro/hunter_steer.xacro (robot description, xacro)
@@ -14,16 +14,17 @@
                 <origin xyz="0 0 0" rpy="0 0 0" />
                 <geometry>
-                    <cylinder radius="${0.04}" length="${0.06}" />
+                    <mesh
+                        filename="package://hunter_se_description/models/meshes/${name}_steer_link.dae" />
                 </geometry>
             </collision>
             <inertial>
-                <mass value="0.5" />
+                <mass value="0.25" />
                 <origin xyz="0 0 0" />
-                <inertia ixx="0.01" ixy="0" ixz="0" iyy="0.01" iyz="0" izz="0.01" />
+                <inertia ixx="0.000105" ixy="0.0" ixz="0.0" iyy="0.00002" iyz="0.0" izz="0.000105" />
             </inertial>
         </link>
         <link name="${name}_wheel_link">
             <visual>
-                <origin xyz="0 0 0.015" rpy="0 0 ${rotation}" />
+                <origin xyz="0 0 0" rpy="0 0 ${rotation}" />
                 <geometry>
                     <mesh filename="package://hunter_se_description/models/meshes/front_wheel.dae" />
@@ -31,19 +32,22 @@
             </visual>
             <collision>
-                <origin xyz="0 0 0" rpy="1.57 0 0" />
+                <!-- <origin xyz="0 0 0" rpy="1.57 0 0" /> -->
+                <origin xyz="0 0 0" rpy="0 0 ${rotation}" />
                 <geometry>
-                    <cylinder radius="${wheel_radius}" length="${wheel_length}" />
+                    <mesh filename="package://hunter_se_description/models/meshes/front_wheel.dae" />
+                    <!-- <cylinder radius="${wheel_radius}" length="${wheel_length}" /> -->
                 </geometry>
             </collision>
             <inertial>
-                <mass value="0.5" />
+                <mass value="1.0" />
                 <origin xyz="0 0 0" />
-                <inertia ixx="0.022" ixy="0" ixz="0" iyy="0.022" iyz="0" izz="0.0378" />
+                <!-- <inertia ixx="0.22" ixy="0.01" ixz="0.01" iyy="0.22" iyz="0.01" izz="0.378" /> -->
+                <inertia ixx="0.006864" ixy="0.0" ixz="0.0" iyy="0.012106" iyz="0.0" izz="0.006864" />
             </inertial>
             <surface>
                 <friction>
                     <ode>
-                        <mu>0.7</mu>
-                        <mu2>0.7</mu2>
+                        <mu>1.0</mu>
+                        <mu2>1.0</mu2>
                     </ode>
                 </friction>
@@ -52,5 +56,5 @@
         <gazebo reference="${name}_wheel_link">
             <mu1 value="1.0" />
-            <mu2 value="2.0" />
+            <mu2 value="1.0" />
             <kp value="10000000.0" />
             <kd value="1.0" />
@@ -64,5 +68,5 @@
                 rpy="0 0 0" />
             <axis xyz="0 0 1" rpy="0 0 0" />
-            <limit lower="${-max_steer}" upper="${max_steer}" effort="10" velocity="4" />
+            <limit lower="${-max_steer}" upper="${max_steer}" effort="100" velocity="4" />
         </joint>
         <joint name="${name}_wheel_joint" type="continuous">

Commit message: Fixed ackermann_odometry

File: hunter_se_description/models/xacro/hunter_gazebo.xacro (robot description, xacro)
@@ -79,4 +79,5 @@
                 <always_on>true</always_on>
                 <update_rate>100</update_rate>
+                <initial_orientation_as_reference>True</initial_orientation_as_reference>
                 <imu>
                     <angular_velocity>

File: hunter_se_description/models/xacro/hunter_motors.xacro (robot description, xacro)
@@ -11,9 +11,7 @@
             </visual>
             <collision>
-                <!-- <origin xyz="0 0 0" rpy="1.57 0 0" /> -->
                 <origin xyz="0 ${reflect * -0.065} 0" rpy="0 0 ${rotation}" />
                 <geometry>
                     <mesh filename="package://hunter_se_description/models/meshes/rear_wheel.dae" />
-                    <!-- <cylinder radius="${wheel_radius}" length="${wheel_length}" /> -->
                 </geometry>
             </collision>
@@ -22,5 +20,4 @@
                 <origin xyz="0 0 0" />
                 <inertia ixx="0.006864" ixy="0.0" ixz="0.0" iyy="0.012106" iyz="0.0" izz="0.006864" />
-                <!-- <inertia ixx="0.22" ixy="0.02" ixz="0.02" iyy="0.22" iyz="0.02" izz="0.378" /> -->
             </inertial>
             <surface>

File: hunter_se_description/models/xacro/hunter_se.xacro (robot description, xacro)
@@ -45,5 +45,4 @@
             <mass value="38" />
             <origin xyz="0.050 0.00 -0.075" />
-            <!-- <inertia ixx="2.0533" ixy="0.0" ixz="0.0" iyy="2.56993" iyz="0.0" izz="0.69606" /> -->
             <inertia ixx="0.65" ixy="0.0" ixz="0.0" iyy="2.75" iyz="0.0" izz="3.0" />
         </inertial>
@@ -58,14 +57,8 @@
     <xacro:hunter_steer name="front_left" reflect="1" rotation="${-pi/2}" />
     <link name="center_steer_link">
-        <!-- <collision>
-            <origin xyz="0 0 0" rpy="0 0 0" />
-            <geometry>
-                <cylinder radius="${0.04}" length="${0.06}" />
-            </geometry>
-        </collision> -->
         <inertial>
             <mass value="0.25" />
             <origin xyz="0 0 0" rpy="0 0 0" />
-            <inertia ixx="0.000105" ixy="0.0" ixz="0.0" iyy="0.00002" iyz="0.0" izz="0.000105" />
+            <inertia ixx="0.000474" ixy="0.0" ixz="0.0" iyy="0.000474" iyz="0.0" izz="0.000625" />
         </inertial>
     </link>
@@ -81,5 +74,5 @@
     <xacro:hunter_motors name="rear_right" reflect="-1" rotation="${-pi/2}" />
     <xacro:hunter_motors name="rear_left" reflect="1" rotation="${pi/2}" />
-    <!-- <xacro:ackermann_odometry /> -->
+    <xacro:ackermann_odometry />
     <xacro:imu name="IMU" parent="base_link" />
     <ros2_control name="GazeboSystem" type="system">

File: hunter_se_description/models/xacro/hunter_steer.xacro (robot description, xacro)
@@ -21,5 +21,5 @@
                 <mass value="0.25" />
                 <origin xyz="0 0 0" />
-                <inertia ixx="0.000105" ixy="0.0" ixz="0.0" iyy="0.00002" iyz="0.0" izz="0.000105" />
+                <inertia ixx="0.000474" ixy="0.0" ixz="0.0" iyy="0.000474" iyz="0.0" izz="0.000625" />
             </inertial>
         </link>
@@ -32,9 +32,7 @@
             </visual>
             <collision>
-                <!-- <origin xyz="0 0 0" rpy="1.57 0 0" /> -->
                 <origin xyz="0 0 0" rpy="0 0 ${rotation}" />
                 <geometry>
                     <mesh filename="package://hunter_se_description/models/meshes/front_wheel.dae" />
-                    <!-- <cylinder radius="${wheel_radius}" length="${wheel_length}" /> -->
                 </geometry>
             </collision>
@@ -42,5 +40,4 @@
                 <mass value="1.0" />
                 <origin xyz="0 0 0" />
-                <!-- <inertia ixx="0.22" ixy="0.01" ixz="0.01" iyy="0.22" iyz="0.01" izz="0.378" /> -->
                 <inertia ixx="0.006864" ixy="0.0" ixz="0.0" iyy="0.012106" iyz="0.0" izz="0.006864" />
             </inertial>
@@ -75,5 +72,4 @@
             <origin xyz="0 ${reflect * steering_wheel_y_offset} ${steering_wheel_z_offset}" />
             <axis xyz="0 1 0" rpy="0 0 0" />
-            <!-- <dynamics damping="0.0" friction="2.0" /> -->
         </joint>
     </xacro:macro>
