Commit message: Added Odometry and RVIZ

File: hunter_se_description/models/xacro/hunter_gazebo.xacro (robot description, xacro)
@@ -45,5 +45,5 @@
                 <left_steering_joint>front_left_steer_joint</left_steering_joint>
                 <right_steering_joint>front_right_steer_joint</right_steering_joint>
-                <steering_wheel_joint>center_steer_joint</steering_wheel_joint>
+                <!-- <steering_wheel_joint>center_steer_joint</steering_wheel_joint> -->
                 <max_steer>0.690</max_steer>
                 <max_speed>15</max_speed>
@@ -58,5 +58,5 @@
                 <publish_wheel_tf>false</publish_wheel_tf>
                 <publish_distance>false</publish_distance>
-                <odometry_frame>wheel_odom</odometry_frame>
+                <odometry_frame>odom</odometry_frame>
                 <robot_base_frame>base_link</robot_base_frame>
             </plugin>
@@ -74,4 +74,5 @@
                 <plugin filename="libgazebo_ros_imu_sensor.so" name="imu_plugin">
                     <ros>
+                        <namespace>${robot_namespace}</namespace>
                         <remapping>~/out:=imu</remapping>
                     </ros>

File: hunter_se_description/models/xacro/hunter_motors.xacro (robot description, xacro)
@@ -17,16 +17,8 @@
             </collision>
             <inertial>
-                <mass value="1.0" />
+                <mass value="2.5" />
                 <origin xyz="0 0 0" />
                 <inertia ixx="0.006864" ixy="0.0" ixz="0.0" iyy="0.012106" iyz="0.0" izz="0.006864" />
             </inertial>
-            <surface>
-                <friction>
-                    <ode>
-                        <mu>1.0</mu>
-                        <mu2>1.0</mu2>
-                    </ode>
-                </friction>
-            </surface>
         </link>
         <joint name="${name}_wheel_joint" type="continuous">
@@ -38,9 +30,11 @@
         </joint>
         <gazebo reference="${name}_wheel_link">
-            <mu1 value="1.0" />
+            <mu1 value="2.0" />
             <mu2 value="1.0" />
             <kp value="10000000.0" />
             <kd value="1.0" />
-            <fdir1 value="0 1 0" />
+            <fdir1 value="1 0 0" />
+            <slip1>0</slip1>
+            <slip2>0</slip2>
         </gazebo>
     </xacro:macro>

File: hunter_se_description/models/xacro/hunter_se.xacro (robot description, xacro)
@@ -43,5 +43,5 @@
         </collision>
         <inertial>
-            <mass value="38" />
+            <mass value="50.0" />
             <origin xyz="0.050 0.00 -0.075" />
             <inertia ixx="0.65" ixy="0.0" ixz="0.0" iyy="2.75" iyz="0.0" izz="3.0" />
@@ -56,20 +56,4 @@
     <xacro:hunter_steer name="front_right" reflect="-1" rotation="${pi/2}" />
     <xacro:hunter_steer name="front_left" reflect="1" rotation="${-pi/2}" />
-    <link name="center_steer_link">
-        <inertial>
-            <mass value="0.25" />
-            <origin xyz="0 0 0" rpy="0 0 0" />
-            <inertia ixx="0.000474" ixy="0.0" ixz="0.0" iyy="0.000474" iyz="0.0" izz="0.000625" />
-        </inertial>
-    </link>
-    <joint name="center_steer_joint" type="revolute">
-        <parent link="base_link" />
-        <child link="center_steer_link" />
-        <origin
-            xyz="${steering_axle_x_offset} 0 ${steering_axle_z_offset}"
-            rpy="0 0 0" />
-        <axis xyz="0 0 1" />
-        <limit lower="${-max_steer}" upper="${max_steer}" effort="100" velocity="5.0" />
-    </joint>
     <xacro:hunter_motors name="rear_right" reflect="-1" rotation="${-pi/2}" />
     <xacro:hunter_motors name="rear_left" reflect="1" rotation="${pi/2}" />
@@ -81,8 +65,4 @@
             <robotNamespace>${robot_namespace}</robotNamespace>
         </hardware>
-        <xacro:steering_control
-            name="center"
-            steer_limlow="${-max_steer}"
-            steer_limhigh="${max_steer}" />
         <xacro:steering_control
             name="front_right"

File: hunter_se_description/models/xacro/hunter_steer.xacro (robot description, xacro)
@@ -38,18 +38,20 @@
             </collision>
             <inertial>
-                <mass value="1.0" />
+                <mass value="2.5" />
                 <origin xyz="0 0 0" />
-                <inertia ixx="0.006864" ixy="0.0" ixz="0.0" iyy="0.012106" iyz="0.0" izz="0.006864" />
+                <!-- <inertia ixx="0.006864" ixy="0.0" ixz="0.0" iyy="0.012106" iyz="0.0" izz="0.006864" /> -->
+                <inertia ixx="0.008064" ixy="0.0" ixz="0.0" iyy="0.012106" iyz="0.0" izz="0.008064" />
             </inertial>
-            <surface>
-                <friction>
-                    <ode>
-                        <mu>1.0</mu>
-                        <mu2>1.0</mu2>
-                    </ode>
-                </friction>
-            </surface>
         </link>
         <gazebo reference="${name}_wheel_link">
+            <mu1 value="2.0" />
+            <mu2 value="1.0" />
+            <kp value="10000000.0" />
+            <kd value="1.0" />
+            <fdir1 value="1 0 0" />
+            <slip1>0</slip1>
+            <slip2>0</slip2>
+        </gazebo>
+        <gazebo reference="${name}_steer_link">
             <mu1 value="1.0" />
             <mu2 value="1.0" />
@@ -57,4 +59,6 @@
             <kd value="1.0" />
             <fdir1 value="0 1 0" />
+            <slip1>0</slip1>
+            <slip2>0</slip2>
         </gazebo>
         <joint name="${name}_steer_joint" type="revolute">
